File: pedals_for_microscope.sch (KiCad schematic (older format))
At the start: 45 parts

Commit message: xcv
Parts:
- removed C?: 12pF, symbol C
- C1, C4, C6, C7: renamed from C?; footprint (none) -> Capacitor_SMD:C_0805_2012Metric
- C10, C11, C12, C14, C15, C17, C18, C19, C20, C21, C5: renamed from C?; footprint (none) -> Capacitor_SMD:C_0402_1005Metric
- C8, C9: renamed from C?; footprint (none) -> Capacitor_SMD:C_0603_1608Metric
- J1, J2, J5: renamed from J?; footprint (none) -> Connectors_Molex:Molex_PicoBlade_53261-0471_04x1.25mm_Angled
- J3, J4, J6, J7: renamed from J?; footprint Connector_PinHeader_2.54mm:PinHeader_1x03_P2.54mm_Vertical -> Connectors_Molex:Molex_PicoBlade_53261-0371_03x1.25mm_Angled
- R1, R2, R3, R4, R5, R6: renamed from R?; footprint (none) -> Resistor_SMD:R_0402_1005Metric
- SW1: renamed from SW?; value SW_Push -> RESET; footprint (none) -> MAR_inductors:EVQPE104K
- U1: renamed from U?; footprint (none) -> MAR_inductors:nRF52840
- gave numbers to parts that had none: 12
Connections:
- no-connect marks 0 -> 45
